Commit message: Added possibility to deactivate transmission (not supported by default ros control and no local RobotHW defined)

File: robots/sensor.urdf.xacro (robot description, xacro)
@@ -4,4 +4,5 @@
   <xacro:arg name="model" default="gamma" />
   <xacro:arg name="sim" default="false" />
+  <xacro:arg name="controller" default="false" />
   <!-- ati sensor -->
   <xacro:include filename="$(find ati_sensor_description)/urdf/ati_sensor.urdf.xacro" />
@@ -9,5 +10,5 @@
   <link name="world"/>
   <!-- sensor -->
-  <xacro:ati_sensor prefix="" child="" model="$(arg model)" sim="$(arg sim)"/>
+  <xacro:ati_sensor prefix="" child="" model="$(arg model)" sim="$(arg sim)" controller="$(arg controller)"/>
   <joint name="ft_base_fixed_joint" type="fixed">
     <origin xyz="0 0 0" rpy="0 0 0" />

File: urdf/ati_sensor.urdf.xacro (robot description, xacro)
@@ -2,5 +2,5 @@
 <robot xmlns:xacro="http://www.ros.org/wiki/xacro"
        name="ati_sensor" >
-  <xacro:macro name="ati_sensor" params="prefix:='' child:='' model:='gamma' interface_height:='-' sim:=false rate:=100">
+  <xacro:macro name="ati_sensor" params="prefix:='' child:='' model:='gamma' interface_height:='-' sim:=false controller:=false rate:=100">
     <!-- access sensor models -->
     <xacro:property name="package_path" value="$(find ati_sensor_description)" />
@@ -62,5 +62,7 @@
       <limit effort="100.0" lower="0.0" upper="0.0001" velocity="100.0"/>
     </joint>
-    <xacro:fts_transmission/>
+    <xacro:if value="${controller}">
+      <xacro:fts_transmission/>
+    </xacro:if>
     <!-- if provided, attach the tool to the ati sensor -->
     <xacro:if value="${1 if child else 0}">
